File: pcb/subpar-drive.sch (EAGLE design)
At the start: 38 parts, among them U1 ATSAME70Q20-LFBGA144, U2 ICE40HX4K-BG121

Commit message: add docu; add fpga
Parts:
- added C21, C22, C23, C24, C25, C26, C27, C28, C29, C30, C31, C32, C33, C34, C35, C36, C37, C38, C39: 100n, Passive Components > Capacitors > Multilayer Ceramic Capacitors MLCC:MLCC_0402
- added C6: 4u7, Passive Components > Capacitors > Multilayer Ceramic Capacitors MLCC:MLCC0603
- added R10, R11, R12, R8: 10k, Passive Components > Resistors > Chip Resistors:RESISTOR_0402
- added R9: 100, Passive Components > Resistors > Chip Resistors:RESISTOR_0402
- added TP1: TEST_POINT, Utility > Board:TEST_POINT
- U2: value ICE40HX4K-BG121 -> ICE40HX8K-CT256; device Semiconductors > Embedded Processors & Controllers > FPGA - Field Programmable Gate Array:ICE40HX4K-BG121 -> Semiconductors > Embedded Processors & Controllers > FPGA - Field Programmable Gate Array:ICE40HX8K-CT256
Connections:
- net VDDCORE renamed VCORE
- new net !FPGA_CRST: R8.P$2, U2.PWRCTRL.!CRESET
- new net !FPGA_SS: R12.P$2, U2.BANK2SPI.!SS!/IOB_108
- new net 1.2V: C22.P$1, C23.P$1, C24.P$1, C25.P$1, C26.P$1, C27.P$1, R9.P$1, U2.PWRCTRL.VCC@0, U2.PWRCTRL.VCC@1, U2.PWRCTRL.VCC@2, U2.PWRCTRL.VCC@3, U2.PWRCTRL.VCC@4, U2.PWRCTRL.VCC@5
- new net FPGA_CBSEL0: U2.BANK2SPI.CBSEL0/IOB_103
- new net FPGA_CBSEL1: U2.BANK2SPI.CBSEL1/IOB_104
- new net FPGA_CDONE: R10.P$1, U2.PWRCTRL.CDONE
- new net FPGA_CLK: U2.BANK0.IOT_198_GBIN0
- new net FPGA_MISO: U2.BANK2SPI.SDO/IOB_105
- new net FPGA_MOSI: U2.BANK2SPI.SDI/IOB_106
- new net FPGA_SCK: R11.P$1, U2.BANK2SPI.SCK/IOB_107
- new net GNDPLL: C21.P$2, C6.P$2
- new net GND_PLL: U2.PWRCTRL.GNDPLL0, U2.PWRCTRL.GNDPLL1
- new net N$12: C21.P$1, C6.P$1, R9.P$2, U2.PWRCTRL.VCCPLL0, U2.PWRCTRL.VCCPLL1
- new net N$13: TP1.S, U2.PWRCTRL.VPP_FAST
- net 3.3V: now also C28.P$1, C29.P$1, C30.P$1, C31.P$1, C32.P$1, C33.P$1, C34.P$1, C35.P$1, C36.P$1, C37.P$1, C38.P$1, C39.P$1, R10.P$2, R11.P$2, U2.PWRCTRL.VCCIO0@0, U2.PWRCTRL.VCCIO0@1, U2.PWRCTRL.VCCIO0@2, U2.PWRCTRL.VCCIO0@3, U2.PWRCTRL.VCCIO1@0, U2.PWRCTRL.VCCIO1@1, U2.PWRCTRL.VCCIO1@2, U2.PWRCTRL.VCCIO1@3, U2.PWRCTRL.VCCIO2@0, U2.PWRCTRL.VCCIO2@1, U2.PWRCTRL.VCCIO2@2, U2.PWRCTRL.VCCIO2@3, U2.PWRCTRL.VCCIO3@0, U2.PWRCTRL.VCCIO3@1, U2.PWRCTRL.VCCIO3@2, U2.PWRCTRL.VCCIO3@3, U2.PWRCTRL.VCC_SPI, U2.PWRCTRL.VPP_2V5
- net GND: now also C22.P$2, C23.P$2, C24.P$2, C25.P$2, C26.P$2, C27.P$2, C28.P$2, C29.P$2, C30.P$2, C31.P$2, C32.P$2, C33.P$2, C34.P$2, C35.P$2, C36.P$2, C37.P$2, C38.P$2, C39.P$2, R12.P$1, R8.P$1, U2.PWRCTRL.GND@0, U2.PWRCTRL.GND@1, U2.PWRCTRL.GND@10, U2.PWRCTRL.GND@11, U2.PWRCTRL.GND@12, U2.PWRCTRL.GND@13, U2.PWRCTRL.GND@14, U2.PWRCTRL.GND@15, U2.PWRCTRL.GND@16, U2.PWRCTRL.GND@17, U2.PWRCTRL.GND@2, U2.PWRCTRL.GND@3, U2.PWRCTRL.GND@4, U2.PWRCTRL.GND@5, U2.PWRCTRL.GND@6, U2.PWRCTRL.GND@7, U2.PWRCTRL.GND@8, U2.PWRCTRL.GND@9
Other:
- note added: "A14"
- note added: "A3"
- note added: "E1"
- note added: "F10"
- note added: "F6"
- note added: "F8"
- note added: "FPGA power and ctrl"
- note added: "H10"
- note added: "J6"
- note added: "K10"
- note added: "K6"
- note added: "L2"
- note added: "N13"
- note added: "N15"
- note added: "P3"
- note added: "R8"

Commit message: added power sheet
Parts:
- added U3: MIC23159, Power > Switching Controllers:MIC23159
- added U4: MIC2253, Power > Switching Controllers:MIC2253
- added U5: MIC24052, Power > Switching Controllers:MIC24052
Changed lines of the file:
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@@
 <?xml version="1.0" encoding="utf-8"?>
 <!DOCTYPE eagle SYSTEM "eagle.dtd">
-<eagle version="9.5.1">
+<eagle version="9.5.0">
 <drawing>
 <settings>
@@
 <part name="R12" library="Passive Components &gt; Resistors &gt; Chip Resistors" deviceset="RESISTOR" device="_0402" value="10k"/>
 <part name="GND24" library="Utility &gt; Power Symbols" deviceset="GND" device=""/>
+<part name="FRAME4" library="Utility &gt; Schematic" deviceset="FRAME" device=""/>
+<part name="U3" library="Power &gt; Switching Controllers" deviceset="MIC23159" device=""/>
+<part name="U4" library="Power &gt; Switching Controllers" deviceset="MIC2253" device=""/>
+<part name="U5" library="Power &gt; Switching Controllers" deviceset="MIC24052" device=""/>
 </parts>
 <sheets>
@@
 </nets>
 </sheet>
+<sheet>
+<description>Power manager</description>
+<plain>
+</plain>
+<instances>
+<instance part="FRAME4" gate="G$1" x="0" y="0" smashed="yes"/>
+<instance part="FRAME4" gate="G$2" x="278.13" y="10.16" smashed="yes">
+<attribute name="LAST_DATE_TIME" x="290.322" y="11.43" size="2.54" layer="94"/>
+<attribute name="SHEET" x="363.474" y="11.43" size="2.54" layer="94"/>
+<attribute name="DESIGNER" x="279.6" y="16.764" size="2.54" layer="94"/>
+<attribute name="CREVISION" x="367" y="17.68" size="2.54" layer="94"/>
+<attribute name="LICENSE" x="280.67" y="5.588" size="2.159" layer="94"/>
+<attribute name="LINK" x="280.67" y="1.778" size="1.778" layer="94"/>
+<attribute name="DRAWING_NAME" x="292.3" y="27.94" size="2.54" layer="94"/>
+<attribute name="COMPANY" x="335.48" y="16.764" size="2.54" layer="94"/>
+</instance>
+<instance part="U3" gate="G$1" x="243.84" y="134.62" smashed="yes">
+<attribute name="NAME" x="213.36" y="138.176" size="1.27" layer="95"/>
+<attribute name="VALUE" x="213.36" y="135.89" size="1.27" layer="96"/>
+</instance>
+<instance part="U4" gate="G$1" x="236.22" y="177.8" smashed="yes">
+<attribute name="NAME" x="215.9" y="181.356" size="1.27" layer="95"/>
+<attribute name="VALUE" x="215.9" y="179.07" size="1.27" layer="96"/>
+</instance>
+<instance part="U5" gate="G$1" x="170.18" y="147.32" smashed="yes">
+<attribute name="NAME" x="142.24" y="150.876" size="1.27" layer="95"/>
+<attribute name="VALUE" x="142.24" y="148.59" size="1.27" layer="96"/>
+</instance>
+</instances>
+<busses>
+</busses>
+<nets>
+</nets>
+</sheet>
